File: hw/sch_pcb/DATALOGGER01A.kicad_pcb (KiCad board)
At the start: 2 copper layers, 80.8 x 101.1 mm, 91 parts, among them J1 HEADER_2x01_PARALLEL, J10 HEADER_2x03_PARALLEL, J11 HEADER_2x01, J12 HEADER_2x01_PARALLEL, J13 HEADER_2x01_PARALLEL, J14 HEADER_2x01_PARALLEL, J15 HEADER_2x01_PARALLEL, J16 HEADER_2x01_PARALLEL, J17 HEADER_2x01_PARALLEL, J18 HEADER_2x01_PARALLEL, J19 HEADER_2x01_PARALLEL, J2 HEADER_2x01_PARALLEL, J20 HEADER_2x01_PARALLEL, J21 HEADER_2x01, J22 HEADER_2x01_PARALLEL, J23 HEADER_2x01_PARALLEL, J24 HEADER_2x01_PARALLEL, J25 HEADER_2x01_PARALLEL, J26 HEADER_2x01_PARALLEL, J27 HEADER_2x01_PARALLEL, J28 HEADER_2x01_PARALLEL, J29 HEADER_2x01_PARALLEL, J3 HEADER_2x01_PARALLEL, J30 HEADER_2x01_PARALLEL, J31 HEADER_2x03, J32 HEADER_2x01, J33 HEADER_2x03_PARALLEL, J34 MCC-SD (kouka z modulu), J4 HEADER_2x01_PARALLEL, J5 HEADER_2x01_PARALLEL, J6 HEADER_2x03_PARALLEL, J7 MCC-SD, J8 HEADER_2x01_PARALLEL, J9 HEADER_2x01, M1 HOLE, M2 HOLE, M3 HOLE, M4 HOLE, SW1 5MS1S102AM6QE, U1 ISL21080CIH320Z-TK, U2 TPS22965-Q1, U3 ATMEGA1284P-AU, U4 PCF85263A, U5 LM4041CIM3-1.2(neosazovat), U6 AT24CS64-SSHM, Y1 16MHz, Y2 ABS07-120-32.768KHZ-T

Commit message: Fix licence and repository cleanup.
Other:
- net class Default removed
- net class MLAB_default removed
- net class MLAB_power removed

Commit message: Update title blocks Place board to the center of page.
Parts:
- removed M1: HOLE, Mlab_Mechanical:MountingHole_3mm
- moved BT1 182.3 mm to (142.4, 77.1)
- moved BT2 182.3 mm to (142.4, 115.2)
- moved BT3 182.3 mm to (143.6, 94.9)
- moved C1 182.3 mm to (135.4, 70.1)
- moved C10 182.3 mm to (163.3, 129.8)
- moved C11 182.3 mm to (142.4, 105.0)
- moved C13 182.3 mm to (165.9, 125.3)
- moved C14 182.3 mm to (146.2, 65.7)
- moved C15 182.3 mm to (142.4, 107.6)
- moved C16 182.3 mm to (177.3, 64.4)
- moved C17 182.3 mm to (148.7, 65.7)
- moved C18 182.3 mm to (170.9, 102.2)
- moved C19 182.3 mm to (163.0, 58.0)
- moved C2 182.3 mm to (137.9, 70.1)
- moved C20 182.3 mm to (166.5, 75.2)
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